File: kicad/keyboard.kicad_sch (KiCad schematic)
At the start: 6 parts, among them SW1 SW_Push, U1 Arduino_pro_Micro

Commit message: Last update
Parts:
- added J1, J2: (no value), symbol Connector:Conn_01x07_Male
Connections:
- net GND: now also J1.1 (Pin_1), J2.1 (Pin_1)
- net SPI_DATA: now also U1.5 (2); no longer U1.8 (5)
- net at U1.10 (7): now also J1.7 (Pin_7)
- net at U1.15 (14): now also J2.3 (Pin_3)
- net at U1.16 (15): now also J2.4 (Pin_4)
- net at U1.17 (18-A0): now also J2.5 (Pin_5)
- net at U1.18 (19-A1): now also J2.6 (Pin_6)
- net at U1.19 (20-A2): now also J2.7 (Pin_7)
- net Vin: now reaches U1.24 (RAW)
- net Vin: now also J1.2 (Pin_2), J2.2 (Pin_2)
- net at U1.6 (3): now also J1.3 (Pin_3)
- net at U1.7 (4): now also J1.4 (Pin_4)
- net at U1.9 (6): now also J1.6 (Pin_6)
- net VCC: no longer names the net of U1.21 (VCC)
- new net: J1.5 (Pin_5), U1.8 (5)
- no-connect marks 14 -> 4
Other:
- moved on the sheet: SW1
