File: kicad/test.kicad_pcb (KiCad board)
At the start: 2 copper layers, 301 x 97.8 mm, 68 parts, among them J1 Conn_01x07_Male, J2 Conn_01x07_Male, SW1 SW_Push, SW10 Gateron_ks_27, SW11 Gateron_ks_27, SW12 Gateron_ks_27, SW13 Gateron_ks_27, SW14 Gateron_ks_27, SW15 Gateron_ks_27, SW16 Gateron_ks_27, SW17 Gateron_ks_27, SW18 Gateron_ks_27, SW19 Gateron_ks_27, SW20 Gateron_ks_27, SW21 Gateron_ks_27, SW22 Gateron_ks_27, SW23 Gateron_ks_27, SW24 Gateron_ks_27, SW25 Gateron_ks_27, SW26 Gateron_ks_27, SW27 Gateron_ks_27, SW28 Gateron_ks_27, SW29 Gateron_ks_27, SW30 Gateron_ks_27, SW31 Gateron_ks_27, SW32 Gateron_ks_27, SW33 Gateron_ks_27, SW34 Gateron_ks_27, SW35 Gateron_ks_27, SW36 Gateron_ks_27, SW37 Gateron_ks_27, SW38 Gateron_ks_27, SW39 Gateron_ks_27, SW4 Gateron_ks_27, SW40 Gateron_ks_27, SW41 Gateron_ks_27, SW42 Gateron_ks_27, SW43 Gateron_ks_27, SW44 Gateron_ks_27, SW45 Gateron_ks_27, SW46 Gateron_ks_27, SW47 Gateron_ks_27, SW48 Gateron_ks_27, SW49 Gateron_ks_27, SW5 Gateron_ks_27, SW50 Gateron_ks_27, SW51 Gateron_ks_27, SW52 Gateron_ks_27, SW53 Gateron_ks_27, SW54 Gateron_ks_27, SW55 Gateron_ks_27, SW56 Gateron_ks_27, SW57 Gateron_ks_27, SW58 Gateron_ks_27, SW59 Gateron_ks_27, SW6 Gateron_ks_27, SW60 Gateron_ks_27, SW61 Gateron_ks_27, SW7 Gateron_ks_27, SW8 Gateron_ks_27, SW9 Gateron_ks_27, U1 Arduino_pro_Micro, U2 74HC595, U3 74HC595

Commit message: Last update
Parts:
- moved J1 30.7 mm to (57.1, 38.1)
- moved J2 30.6 mm to (285.8, 38.1)
Routing:
- net Vin: track 178.8 -> 239.3 mm
- net Net-(J1-Pad3): track 93.7 -> 123.8 mm
- net Net-(J1-Pad7): track 120.1 -> 149.0 mm
- net Net-(J1-Pad4): track 100.3 -> 129.2 mm
- net Net-(J1-Pad5): track 106.9 -> 135.8 mm
- net Net-(J1-Pad6): track 113.5 -> 142.4 mm
- net Net-(J2-Pad3): track 116.4 -> 145.2 mm
- net Net-(J2-Pad7): track 88.7 -> 117.5 mm
- net Net-(J2-Pad6): track 95.9 -> 124.8 mm
- net Net-(J2-Pad5): track 102.6 -> 131.4 mm
- net Net-(J2-Pad4): track 109.6 -> 138.4 mm
Other:
- board size 301 x 97.8 mm -> 301.6 x 116.8 mm
