File: kicad/keyboard.kicad_pcb (KiCad board)
At the start: 2 copper layers, 301 x 97.8 mm, 68 parts, among them J1 Conn_01x07_Male, J2 Conn_01x07_Male, SW1 SW_Push, SW10 Gateron_ks_27, SW11 Gateron_ks_27, SW12 Gateron_ks_27, SW13 Gateron_ks_27, SW14 Gateron_ks_27, SW15 Gateron_ks_27, SW16 Gateron_ks_27, SW17 Gateron_ks_27, SW18 Gateron_ks_27, SW19 Gateron_ks_27, SW20 Gateron_ks_27, SW21 Gateron_ks_27, SW22 Gateron_ks_27, SW23 Gateron_ks_27, SW24 Gateron_ks_27, SW25 Gateron_ks_27, SW26 Gateron_ks_27, SW27 Gateron_ks_27, SW28 Gateron_ks_27, SW29 Gateron_ks_27, SW30 Gateron_ks_27, SW31 Gateron_ks_27, SW32 Gateron_ks_27, SW33 Gateron_ks_27, SW34 Gateron_ks_27, SW35 Gateron_ks_27, SW36 Gateron_ks_27, SW37 Gateron_ks_27, SW38 Gateron_ks_27, SW39 Gateron_ks_27, SW4 Gateron_ks_27, SW40 Gateron_ks_27, SW41 Gateron_ks_27, SW42 Gateron_ks_27, SW43 Gateron_ks_27, SW44 Gateron_ks_27, SW45 Gateron_ks_27, SW46 Gateron_ks_27, SW47 Gateron_ks_27, SW48 Gateron_ks_27, SW49 Gateron_ks_27, SW5 Gateron_ks_27, SW50 Gateron_ks_27, SW51 Gateron_ks_27, SW52 Gateron_ks_27, SW53 Gateron_ks_27, SW54 Gateron_ks_27, SW55 Gateron_ks_27, SW56 Gateron_ks_27, SW57 Gateron_ks_27, SW58 Gateron_ks_27, SW59 Gateron_ks_27, SW6 Gateron_ks_27, SW60 Gateron_ks_27, SW61 Gateron_ks_27, SW7 Gateron_ks_27, SW8 Gateron_ks_27, SW9 Gateron_ks_27, U1 Arduino_pro_Micro, U2 74HC595, U3 74HC595

Commit message: Update switch diode
Connections:
- U3 pad 7: COL16 -> unconnected-(U3-QH-Pad7)
Routing:
- net ROW2: track 310.9 -> 314.9 mm
- net Net-(SW15-A): track 3.90 -> 0.00 mm
- net Vin: track 178.8 -> 182.5 mm
- net COL9: track 90.9 -> 94.3 mm
- net ROW1: track 304.2 -> 307.4 mm
- net ROW4: track 372.6 -> 369.5 mm, vias 0 -> 1
- net CLK: track 85.2 -> 87.9 mm
- net Net-(J1-Pin_7): track 120.1 -> 121.9 mm
- net Net-(J1-Pin_6): track 113.5 -> 115.1 mm
- net Net-(J1-Pin_5): track 106.9 -> 108.3 mm
- net Net-(J2-Pin_7): track 88.7 -> 90.1 mm
- net ROW3: track 350.4 -> 351.7 mm, vias 0 -> 1
- net Net-(J2-Pin_5): track 102.6 -> 103.8 mm
- net Net-(J2-Pin_4): track 109.6 -> 110.8 mm
- net Net-(J1-Pin_4): track 100.3 -> 101.5 mm
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
Commit message: Update PCB
Parts:
- added D1: 1N4148W, Diode_SMD:D_SOD-123, F.Cu at (29.3, 59.7)
- added D10: 1N4148W, Diode_SMD:D_SOD-123, F.Cu at (65.5, 83.3)
- added D11: 1N4148W, Diode_SMD:D_SOD-123, F.Cu at (84.3, 83.1)
- added D12: 1N4148W, Diode_SMD:D_SOD-123, F.Cu at (103.6, 80.5)
- added D13: 1N4148W, Diode_SMD:D_SOD-123, F.Cu at (122.2, 87.4)
- added D14: 1N4148W, Diode_SMD:D_SOD-123, F.Cu at (141.2, 89.7)
- added D15: 1N4148W, Diode_SMD:D_SOD-123, F.Cu at (163.8, 108.5)
- added D16: 1N4148W, Diode_SMD:D_SOD-123, F.Cu at (24.9, 97.5)
- added D17: 1N4148W, Diode_SMD:D_SOD-123, F.Cu at (43.9, 100.1)
- added D18: 1N4148W, Diode_SMD:D_SOD-123, F.Cu at (63.0, 101.9)
- added D19: 1N4148W, Diode_SMD:D_SOD-123, F.Cu at (82.0, 101.9)
- added D2: 1N4148W, Diode_SMD:D_SOD-123, F.Cu at (48.3, 62.2)
- added D20: 1N4148W, Diode_SMD:D_SOD-123, F.Cu at (101.6, 99.3)
- added D21: 1N4148W, Diode_SMD:D_SOD-123, F.Cu at (119.6, 106.7)
- added D22: 1N4148W, Diode_SMD:D_SOD-123, F.Cu at (138.7, 109.0)
- added D23: 1N4148W, Diode_SMD:D_SOD-123, F.Cu at (164.1, 128.8)
- added D24: 1N4148W, Diode_SMD:D_SOD-123, F.Cu at (22.4, 116.6)
- added D25: 1N4148W, Diode_SMD:D_SOD-123, F.Cu at (41.7, 118.6)
- added D26: 1N4148W, Diode_SMD:D_SOD-123, F.Cu at (60.2, 121.2)
- added D27: 1N4148W, Diode_SMD:D_SOD-123, F.Cu at (79.5, 121.2)
- added D28: 1N4148W, Diode_SMD:D_SOD-123, F.Cu at (99.3, 117.9)
- added D29: 1N4148W, Diode_SMD:D_SOD-123, F.Cu at (117.6, 125.7)
- added D3: 1N4148W, Diode_SMD:D_SOD-123, F.Cu at (67.3, 64.3)
- added D30: 1N4148W, Diode_SMD:D_SOD-123, F.Cu at (136.4, 128.0)
- added D31: 1N4148W, Diode_SMD:D_SOD-123, F.Cu at (185.2, 71.1)
- added D32: 1N4148W, Diode_SMD:D_SOD-123, F.Cu at (203.5, 68.8)
- added D33: 1N4148W, Diode_SMD:D_SOD-123, F.Cu at (222.0, 61.5)
- added D34: 1N4148W, Diode_SMD:D_SOD-123, F.Cu at (241.3, 64.3)
- added D35: 1N4148W, Diode_SMD:D_SOD-123, F.Cu at (260.6, 64.3)
- added D36: 1N4148W, Diode_SMD:D_SOD-123, F.Cu at (279.7, 62.2)
- added D37: 1N4148W, Diode_SMD:D_SOD-123, F.Cu at (298.2, 59.9)
- added D38: 1N4148W, Diode_SMD:D_SOD-123, F.Cu at (186.9, 90.2)
- added D39: 1N4148W, Diode_SMD:D_SOD-123, F.Cu at (206.2, 87.6)
- added D4: 1N4148W, Diode_SMD:D_SOD-123, F.Cu at (86.9, 64.0)
- added D40: 1N4148W, Diode_SMD:D_SOD-123, F.Cu at (224.3, 80.5)
- added D41: 1N4148W, Diode_SMD:D_SOD-123, F.Cu at (243.8, 83.1)
- added D42: 1N4148W, Diode_SMD:D_SOD-123, F.Cu at (262.9, 83.3)
- added D43: 1N4148W, Diode_SMD:D_SOD-123, F.Cu at (281.9, 80.8)
- added D44: 1N4148W, Diode_SMD:D_SOD-123, F.Cu at (300.7, 78.7)
- added D45: 1N4148W, Diode_SMD:D_SOD-123, F.Cu at (189.5, 109.0)
- added D46: 1N4148W, Diode_SMD:D_SOD-123, F.Cu at (208.3, 106.7)
- added D47: 1N4148W, Diode_SMD:D_SOD-123, F.Cu at (226.6, 99.3)
- added D48: 1N4148W, Diode_SMD:D_SOD-123, F.Cu at (246.4, 102.4)
- added D49: 1N4148W, Diode_SMD:D_SOD-123, F.Cu at (265.4, 102.1)
- added D5: 1N4148W, Diode_SMD:D_SOD-123, F.Cu at (106.2, 61.5)
- added D50: 1N4148W, Diode_SMD:D_SOD-123, F.Cu at (284.5, 99.8)
- added D51: 1N4148W, Diode_SMD:D_SOD-123, F.Cu at (303.3, 97.5)
- added D52: 1N4148W, Diode_SMD:D_SOD-123, F.Cu at (191.8, 127.8)
- added D53: 1N4148W, Diode_SMD:D_SOD-123, F.Cu at (210.6, 125.5)
- added D54: 1N4148W, Diode_SMD:D_SOD-123, F.Cu at (229.1, 118.1)
- added D55: 1N4148W, Diode_SMD:D_SOD-123, F.Cu at (248.4, 120.9)
- added D56: 1N4148W, Diode_SMD:D_SOD-123, F.Cu at (267.7, 121.2)
- added D57: 1N4148W, Diode_SMD:D_SOD-123, F.Cu at (286.5, 118.9)
- added D58: 1N4148W, Diode_SMD:D_SOD-123, F.Cu at (305.6, 116.6)
- added D59: LED, LED_SMD:LED_0805_2012Metric, F.Cu at (176.5, 44.2)
- added D6: 1N4148W, Diode_SMD:D_SOD-123, F.Cu at (124.5, 68.8)
- added D7: 1N4148W, Diode_SMD:D_SOD-123, F.Cu at (143.3, 71.1)
- added D8: 1N4148W, Diode_SMD:D_SOD-123, F.Cu at (27.2, 78.7)
- added D9: 1N4148W, Diode_SMD:D_SOD-123, F.Cu at (46.2, 81.0)
- added R5: 220R, Resistor_SMD:R_0603_1608Metric, F.Cu at (176.3, 48.8)
- J1: footprint Keyboard:PinHeader_01x07 -> Connector_PinHeader_2.54mm:PinHeader_1x05_P2.54mm_Vertical
- R1, R2, R3, R4: footprint Resistor_THT:R_Axial_DIN0207_L6.3mm_D2.5mm_P7.62mm_Horizontal -> Resistor_SMD:R_0603_1608Metric
- moved R3 16.7 mm to (156.2, 82.5)
- moved R4 16.5 mm to (156.2, 85.3)
- moved R2 5.48 mm to (156.2, 79.8), turned to 180 degrees
- moved R1 3.07 mm to (156.2, 77.2), turned to 180 degrees
Connections:
- J2 pad 3: Net-(J2-Pin_3) -> ~{RST}
- J2 pad 4: Net-(J2-Pin_4) -> MOSI
- J2 pad 5: Net-(J2-Pin_5) -> MISO
- J2 pad 6: Net-(J2-Pin_6) -> SCLK
- SW10 pad 1: Net-(SW10-A) -> Net-(D2-A)
- SW11 pad 1: Net-(SW11-A) -> Net-(D9-A)
- SW12 pad 1: Net-(SW12-A) -> Net-(D17-A)
- SW13 pad 1: Net-(SW13-A) -> Net-(D25-A)
- SW14 pad 1: Net-(SW14-A) -> Net-(D3-A)
- SW15 pad 1: Net-(SW15-A) -> Net-(D10-A)
- SW16 pad 1: Net-(SW16-A) -> Net-(D18-A)
- SW17 pad 1: Net-(SW17-A) -> Net-(D26-A)
- SW18 pad 1: Net-(SW18-A) -> Net-(D4-A)
- SW19 pad 1: Net-(SW19-A) -> Net-(D11-A)
- SW20 pad 1: Net-(SW20-A) -> Net-(D19-A)
- SW21 pad 1: Net-(SW21-A) -> Net-(D27-A)
- SW22 pad 1: Net-(SW22-A) -> Net-(D5-A)
- SW23 pad 1: Net-(SW23-A) -> Net-(D12-A)
- SW24 pad 1: Net-(SW24-A) -> Net-(D20-A)
- SW25 pad 1: Net-(SW25-A) -> Net-(D28-A)
- SW26 pad 1: Net-(SW26-A) -> Net-(D6-A)
- SW27 pad 1: Net-(SW27-A) -> Net-(D13-A)
- SW28 pad 1: Net-(SW28-A) -> Net-(D21-A)
- SW29 pad 1: Net-(SW29-A) -> Net-(D29-A)
- SW30 pad 1: Net-(SW30-A) -> Net-(D7-A)
- SW31 pad 1: Net-(SW31-A) -> Net-(D14-A)
- SW32 pad 1: Net-(SW32-A) -> Net-(D22-A)
- SW33 pad 1: Net-(SW33-A) -> Net-(D30-A)
- SW34 pad 1: Net-(SW34-A) -> Net-(D31-A)
- SW35 pad 1: Net-(SW35-A) -> Net-(D38-A)
- SW36 pad 1: Net-(SW36-A) -> Net-(D45-A)
- SW37 pad 1: Net-(SW37-A) -> Net-(D52-A)
- SW38 pad 1: Net-(SW38-A) -> Net-(D32-A)
- SW39 pad 1: Net-(SW39-A) -> Net-(D39-A)
- SW4 pad 1: Net-(SW4-A) -> Net-(D15-A)
- SW40 pad 1: Net-(SW40-A) -> Net-(D46-A)
- SW41 pad 1: Net-(SW41-A) -> Net-(D53-A)
- SW42 pad 1: Net-(SW42-A) -> Net-(D33-A)
- SW43 pad 1: Net-(SW43-A) -> Net-(D40-A)
- SW44 pad 1: Net-(SW44-A) -> Net-(D47-A)
- SW45 pad 1: Net-(SW45-A) -> Net-(D54-A)
- SW46 pad 1: Net-(SW46-A) -> Net-(D34-A)
- SW47 pad 1: Net-(SW47-A) -> Net-(D41-A)
- SW48 pad 1: Net-(SW48-A) -> Net-(D48-A)
- SW49 pad 1: Net-(SW49-A) -> Net-(D55-A)
- SW5 pad 1: Net-(SW5-A) -> Net-(D23-A)
- SW50 pad 1: Net-(SW50-A) -> Net-(D35-A)
- SW51 pad 1: Net-(SW51-A) -> Net-(D42-A)
- SW52 pad 1: Net-(SW52-A) -> Net-(D49-A)
- SW53 pad 1: Net-(SW53-A) -> Net-(D56-A)
- SW54 pad 1: Net-(SW54-A) -> Net-(D36-A)
- SW55 pad 1: Net-(SW55-A) -> Net-(D43-A)
- SW56 pad 1: Net-(SW56-A) -> Net-(D50-A)
- SW57 pad 1: Net-(SW57-A) -> Net-(D57-A)
- SW58 pad 1: Net-(SW58-A) -> Net-(D37-A)
- SW59 pad 1: Net-(SW59-A) -> Net-(D44-A)
- SW6 pad 1: Net-(SW6-A) -> Net-(D1-A)
- SW60 pad 1: Net-(SW60-A) -> Net-(D51-A)
- SW61 pad 1: Net-(SW61-A) -> Net-(D58-A)
- SW7 pad 1: Net-(SW7-A) -> Net-(D8-A)
- SW8 pad 1: Net-(SW8-A) -> Net-(D16-A)
- SW9 pad 1: Net-(SW9-A) -> Net-(D24-A)
- U1 pad 10: Net-(J1-Pin_7) -> ROW2
- U1 pad 11: ROW1 -> ROW3
- U1 pad 12: ROW2 -> ROW4
- U1 pad 13: ROW4 -> Net-(U1-10)
- U1 pad 14: ROW3 -> MOSI
- U1 pad 15: Net-(J2-Pin_3) -> MISO
- U1 pad 16: Net-(J2-Pin_4) -> SCLK
- U1 pad 17: Net-(J2-Pin_5) -> unconnected-(U1-18-A0-Pad17)
- U1 pad 18: Net-(J2-Pin_6) -> unconnected-(U1-19-A1-Pad18)
- U1 pad 9: Net-(J1-Pin_6) -> ROW1
Routing:
- net Net-(J1-Pin_7): track 121.9 -> 0.00 mm
- net Net-(J2-Pin_3): track 117.6 -> 0.00 mm
- net Net-(J1-Pin_6): track 115.1 -> 0.00 mm
- net Net-(J2-Pin_4): track 110.8 -> 0.00 mm
- net Net-(J2-Pin_5): track 103.8 -> 0.00 mm
- net Net-(J2-Pin_6): track 96.9 -> 0.00 mm
- net MOSI: track 0.00 -> 89.0 mm
- net MISO: track 0.00 -> 84.8 mm
- net ~{RST}: track 22.2 -> 106.4 mm
- net SCLK: track 0.00 -> 80.7 mm
- net Net-(U1-10): track 0.00 -> 27.6 mm
- net ROW2: track 314.9 -> 327.4 mm
- net ROW4: track 369.5 -> 380.3 mm, vias 1 -> 2
- net ROW1: track 307.4 -> 313.6 mm
- net ROW3: track 351.7 -> 356.6 mm, vias 1 -> 2
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Other:
- outline, holes or cut-outs redrawn
- board text added: "3"
- board text added: "4"
- board text added: "5"
- board text added: "A2"
- board text added: "MISO"
- board text added: "MOSI"
- board text added: "SCLK"
- board text added: "~{RST}"
- board text removed: "A"
- board text removed: "K"
- board text removed: "ROW1"
- board text removed: "ROW2"
- board text removed: "ROW3"
- board text removed: "ROW4"

Commit message: SIPO is SMT
Parts:
- added C2: 10uF, Capacitor_SMD:C_0603_1608Metric, F.Cu at (186.4, 41.4)
- added C3: 10uF, Capacitor_SMD:C_0603_1608Metric, F.Cu at (126.5, 41.9)
- U2, U3: footprint Package_DIP:DIP-16_W7.62mm_Socket -> Package_SO:SO-16_3.9x9.9mm_P1.27mm
- moved U2 13.6 mm to (134.1, 44.5), turned to 90 degrees
- moved U3 5.73 mm to (193.7, 44.4), turned to 90 degrees
Routing:
- net COL2: track 162.1 -> 173.0 mm, vias 0 -> 1
- net COL3: track 148.9 -> 157.4 mm, vias 0 -> 1
- net COL4: track 133.1 -> 140.5 mm, vias 0 -> 1
- net SPI_DATA: track 37.1 -> 29.8 mm
- net CLK: track 87.9 -> 80.7 mm, vias 0 -> 1
- net COL15: track 156.5 -> 163.2 mm, vias 0 -> 1
- net COL5: track 115.2 -> 121.4 mm, vias 0 -> 1
- net Vin: track 183.6 -> 189.7 mm, vias 0 -> 2
- net COL14: track 143.7 -> 149.0 mm, vias 0 -> 1
- net COL1: track 110.2 -> 104.9 mm, vias 0 -> 1
- net COL6: track 91.9 -> 96.7 mm, vias 0 -> 1
- net COL13: track 128.9 -> 133.4 mm, vias 0 -> 1
- net COL7: track 81.9 -> 85.6 mm, vias 0 -> 1
- net COL12: track 106.4 -> 110.0 mm, vias 0 -> 1
- net COL11: track 88.4 -> 91.4 mm, vias 0 -> 1
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